Commit message: noop

File: urdf/Adv_Robotics_Car.xacro (robot description, xacro)
@@ -164,5 +164,5 @@
  </joint>
  <joint name="hokuyo_joint" type="fixed">
-   <origin xyz="0 0 0.185" rpy="0 0 0"/>
+   <origin xyz="0 0 0.1" rpy="0 0 0"/>
    <parent link="base_link"/>
    <child link="hokuyo_link"/>

Commit message: add mybot_laser_filter.cpp

File: urdf/Adv_Robotics_Car.xacro (robot description, xacro)
@@ -164,5 +164,5 @@
  </joint>
  <joint name="hokuyo_joint" type="fixed">
-   <origin xyz="0 0 0.1" rpy="0 0 0"/>
+   <origin xyz="0 0 0.2" rpy="0 0 0"/>
    <parent link="base_link"/>
    <child link="hokuyo_link"/>

Commit message: rename mybot_laser_filter and add mybot_laser_obstacle_clearing_filter

File: urdf/Adv_Robotics_Car.xacro (robot description, xacro)
@@ -132,7 +132,7 @@
     </visual>
     <inertial>
-      <mass value="1e-5" />
+      <mass value="0.1" />
       <origin xyz="0 0 0" rpy="0 0 0"/>
-      <inertia ixx="1e-6" ixy="0" ixz="0" iyy="1e-6" iyz="0" izz="1e-6" />
+      <inertia ixx="0.2" ixy="0" ixz="0" iyy="0.2" iyz="0" izz="0.3" />
     </inertial>
   </link>
@@ -185,20 +185,22 @@
   <!-- hokuyo -->
   <gazebo reference="hokuyo_link">
+    <mu1>1.0</mu1>
+    <mu2>1.0</mu2>
     <sensor type="ray" name="head_hokuyo_sensor">
       <pose>0 0 0 0 0 0</pose>
       <visualize>true</visualize>
-      <update_rate>10</update_rate>
+      <update_rate>5</update_rate>
       <ray>
         <scan>
           <horizontal>
-            <samples>360</samples>
+            <samples>180</samples>
             <resolution>1</resolution>
-            <min_angle>-3.1415927</min_angle>
-            <max_angle>3.1415927</max_angle>
+            <min_angle>-1.57</min_angle>
+            <max_angle>1.57</max_angle>
           </horizontal>
         </scan>
         <range>
           <min>0.10</min>
-          <max>30.0</max>
+          <max>6.0</max>
           <resolution>0.01</resolution>
         </range>
@@ -210,5 +212,5 @@
                reading. -->
           <mean>0.0</mean>
-          <stddev>0.01</stddev>
+          <stddev>0.0</stddev>
         </noise>
       </ray>
